File: DifferentialProbe.sch (KiCad schematic (older format))
At the start: 58 parts, among them J10 Conn_01x01, J11 Conn_01x01, J12 Conn_01x01, J13 Conn_01x01, J16 Conn_01x01, J17 Conn_01x01, J18 Conn_Coaxial, J6 Conn_01x01, J7 Conn_01x01, Q10 BFP740, Q11 BFP740, Q12 BFP740, Q13 BFP740, Q14 BFP740, Q15 BFP740, Q9 BFP740, U5 KA78M05_TO252

Commit message: Cleaned up the layout
Parts:
- R43, R44: value 22R -> 100R; LCSC C25092 -> C25076
Changed lines of the file:
@@
 P 1550 3950
 F 0 "R43" V 1650 3950 50  0000 C CNN
-F 1 "22R" V 1550 3950 50  0000 C CNN
+F 1 "100R" V 1550 3950 50  0000 C CNN
 F 2 "Resistors_SMD:R_0402_NoSilk" V 1480 3950 50  0001 C CNN
 F 3 "" H 1550 3950 50  0001 C CNN
-F 4 "C25092" V 1550 3950 60  0001 C CNN "LCSC"
+F 4 "C25076" V 1550 3950 60  0001 C CNN "LCSC"
 	1    1550 3950
 	0    1    1    0
@@
 P 1550 5850
 F 0 "R44" V 1650 5850 50  0000 C CNN
-F 1 "22R" V 1550 5850 50  0000 C CNN
+F 1 "100R" V 1550 5850 50  0000 C CNN
 F 2 "Resistors_SMD:R_0402_NoSilk" V 1480 5850 50  0001 C CNN
 F 3 "" H 1550 5850 50  0001 C CNN
-F 4 "C25092" V 1550 5850 60  0001 C CNN "LCSC"
+F 4 "C25076" V 1550 5850 60  0001 C CNN "LCSC"
 	1    1550 5850
 	0    1    1    0
