File: Mixer.sch (KiCad schematic (older format))
At the start: 90 parts, among them J100 Conn_01x01, J101 Conn_01x01, J126 Conn_Coaxial, J127 Conn_Coaxial, J128 Conn_01x01, J129 Conn_01x01, J130 Conn_01x01, J131 Conn_01x01, J22 Barrel_Jack, J23 Barrel_Jack, J93 Conn_Coaxial, J95 Conn_Coaxial, J96 Conn_Coaxial, J98 Conn_01x01, J99 Conn_01x01, Q16 BFP740, Q17 BFP740, Q18 BFP740, Q19 BFP740, Q23 BFP740, Q26 BFP740, Q27 BFP740, Q28 BFP740, U3 LM78M05_TO252, U4 LM78M05_TO252

Commit message: Cleaned up the layout
Parts:
- C51: value 15 pF -> 1 pF; LCSC C1548 -> C14971
- R105: value 22R -> 10R
- R106, R80, R90: value 22R -> 47R; LCSC C25077 -> C25118
- R74: LCSC C25077 -> C25092
Changed lines of the file:
@@
 P 3200 3250
 F 0 "R80" V 3300 3250 50  0000 C CNN
-F 1 "22R" V 3200 3250 50  0000 C CNN
+F 1 "47R" V 3200 3250 50  0000 C CNN
 F 2 "Resistors_SMD:R_0402_NoSilk" V 3130 3250 50  0001 C CNN
 F 3 "" H 3200 3250 50  0001 C CNN
-F 4 " C25077" V 3200 3250 60  0001 C CNN "LCSC"
+F 4 "C25118" V 3200 3250 60  0001 C CNN "LCSC"
 	1    3200 3250
 	0    1    1    0
@@
 P 4450 6800
 F 0 "R105" V 4530 6800 50  0000 C CNN
-F 1 "22R" V 4450 6800 50  0000 C CNN
+F 1 "10R" V 4450 6800 50  0000 C CNN
 F 2 "Resistors_SMD:R_0402_NoSilk" V 4380 6800 50  0001 C CNN
 F 3 "" H 4450 6800 50  0001 C CNN
@@
 P 4900 6100
 F 0 "R106" V 4980 6100 50  0000 C CNN
-F 1 "22R" V 4900 6100 50  0000 C CNN
+F 1 "47R" V 4900 6100 50  0000 C CNN
 F 2 "Resistors_SMD:R_0402_NoSilk" V 4830 6100 50  0001 C CNN
 F 3 "" H 4900 6100 50  0001 C CNN
-F 4 " C25077" V 4900 6100 60  0001 C CNN "LCSC"
+F 4 "C25118" V 4900 6100 60  0001 C CNN "LCSC"
 	1    4900 6100
 	0    1    1    0
@@
 P 2950 6400
 F 0 "R90" V 3030 6400 50  0000 C CNN
-F 1 "22R" V 2950 6400 50  0000 C CNN
+F 1 "47R" V 2950 6400 50  0000 C CNN
 F 2 "Resistors_SMD:R_0402_NoSilk" V 2880 6400 50  0001 C CNN
 F 3 "" H 2950 6400 50  0001 C CNN
-F 4 " C25077" V 2950 6400 60  0001 C CNN "LCSC"
+F 4 "C25118" V 2950 6400 60  0001 C CNN "LCSC"
 	1    2950 6400
 	0    -1   -1   0
@@
 P 4700 6800
 F 0 "C51" H 4710 6870 50  0000 L CNN
-F 1 "15 pF" V 4550 6700 50  0000 L CNN
+F 1 "1 pF" V 4550 6700 50  0000 L CNN
 F 2 "Capacitors_SMD:C_0402_NoSilk" H 4700 6800 50  0001 C CNN
 F 3 "" H 4700 6800 50  0001 C CNN
-F 4 "C1548" H 4700 6800 60  0001 C CNN "LCSC"
+F 4 "C14971" H 4700 6800 60  0001 C CNN "LCSC"
 	1    4700 6800
 	-1   0    0    1
@@
 F 2 "Resistors_SMD:R_0402_NoSilk" V 5380 3900 50  0001 C CNN
 F 3 "" H 5450 3900 50  0001 C CNN
-F 4 " C25077" V 5450 3900 60  0001 C CNN "LCSC"
+F 4 "C25092" V 5450 3900 60  0001 C CNN "LCSC"
 	1    5450 3900
 	-1   0    0    1
