File: RFUtilityKnife.sch (KiCad schematic (older format))
At the start: 106 parts, among them J1 Conn_01x01, J14 Conn_01x01, J15 Conn_01x01, J2 Barrel_Jack, J24 Conn_Coaxial, J25 Conn_Coaxial, J26 Conn_01x01, J27 Conn_01x01, J28 Conn_01x01, J29 Conn_01x01, J3 Conn_Coaxial, J30 Conn_01x01, J31 Conn_01x01, J32 Conn_01x01, J33 Conn_01x01, J44 Conn_01x01, J45 Conn_01x01, J48 Conn_01x01, J49 Conn_01x01, J5 Conn_01x01, J53 Conn_01x01, J59 Conn_01x01, J60 Conn_01x01, J63 Conn_01x01, J65 Conn_01x01, J70 Conn_01x01, J71 Conn_01x01, J72 Conn_01x01, J8 Conn_01x01, J9 Conn_01x01, Q1 BFP740, Q2 BFP740, Q3 BFP740, Q4 BFP740, Q5 BFP740, Q6 BFP740, Q7 BFP740, U1 KA78M05_TO252, U6 KA78M05_TO252

Commit message: Cleaned up the layout
Parts:
- C13: value 10 nF -> 1 nF; LCSC C15195 -> C1523
- C50, C52: value 15 pF -> 1 pF; LCSC C1548 -> C14971
- R10, R22, R31: value 22R -> 47R; LCSC C25092 -> C25118
- R2: value 22R -> 100R; LCSC C25092 -> C25076
- R29, R9: value 22R -> 10R; LCSC C25092 -> C25077
Changed lines of the file:
@@
 P 3800 7050
 F 0 "R9" V 3880 7050 50  0000 C CNN
-F 1 "22R" V 3800 7050 50  0000 C CNN
+F 1 "10R" V 3800 7050 50  0000 C CNN
 F 2 "Resistors_SMD:R_0402_NoSilk" V 3730 7050 50  0001 C CNN
 F 3 "" H 3800 7050 50  0001 C CNN
-F 4 "C25092" V 3800 7050 60  0001 C CNN "LCSC"
+F 4 " C25077" V 3800 7050 60  0001 C CNN "LCSC"
 	1    3800 7050
 	-1   0    0    1
@@
 P 1850 6400
 F 0 "R2" V 1950 6400 50  0000 C CNN
-F 1 "22R" V 1850 6400 50  0000 C CNN
+F 1 "100R" V 1850 6400 50  0000 C CNN
 F 2 "Resistors_SMD:R_0402_NoSilk" V 1780 6400 50  0001 C CNN
 F 3 "" H 1850 6400 50  0001 C CNN
-F 4 "C25092" V 1850 6400 60  0001 C CNN "LCSC"
+F 4 "C25076" V 1850 6400 60  0001 C CNN "LCSC"
 	1    1850 6400
 	0    1    1    0
@@
 P 4250 6350
 F 0 "R10" V 4330 6350 50  0000 C CNN
-F 1 "22R" V 4250 6350 50  0000 C CNN
+F 1 "47R" V 4250 6350 50  0000 C CNN
 F 2 "Resistors_SMD:R_0402_NoSilk" V 4180 6350 50  0001 C CNN
 F 3 "" H 4250 6350 50  0001 C CNN
-F 4 "C25092" V 4250 6350 60  0001 C CNN "LCSC"
+F 4 "C25118" V 4250 6350 60  0001 C CNN "LCSC"
 	1    4250 6350
 	0    1    1    0
@@
 P 3250 3950
 F 0 "R29" V 3330 3950 50  0000 C CNN
-F 1 "22R" V 3250 3950 50  0000 C CNN
+F 1 "10R" V 3250 3950 50  0000 C CNN
 F 2 "Resistors_SMD:R_0402_NoSilk" V 3180 3950 50  0001 C CNN
 F 3 "" H 3250 3950 50  0001 C CNN
-F 4 "C25092" V 3250 3950 60  0001 C CNN "LCSC"
+F 4 " C25077" V 3250 3950 60  0001 C CNN "LCSC"
 	1    3250 3950
 	-1   0    0    1
@@
 P 1850 3550
 F 0 "R22" V 1930 3550 50  0000 C CNN
-F 1 "22R" V 1850 3550 50  0000 C CNN
+F 1 "47R" V 1850 3550 50  0000 C CNN
 F 2 "Resistors_SMD:R_0402_NoSilk" V 1780 3550 50  0001 C CNN
 F 3 "" H 1850 3550 50  0001 C CNN
-F 4 "C25092" V 1850 3550 60  0001 C CNN "LCSC"
+F 4 "C25118" V 1850 3550 60  0001 C CNN "LCSC"
 	1    1850 3550
 	0    1    1    0
@@
 P 3700 3250
 F 0 "R31" V 3780 3250 50  0000 C CNN
-F 1 "22R" V 3700 3250 50  0000 C CNN
+F 1 "47R" V 3700 3250 50  0000 C CNN
 F 2 "Resistors_SMD:R_0402_NoSilk" V 3630 3250 50  0001 C CNN
 F 3 "" H 3700 3250 50  0001 C CNN
-F 4 "C25092" V 3700 3250 60  0001 C CNN "LCSC"
+F 4 "C25118" V 3700 3250 60  0001 C CNN "LCSC"
 	1    3700 3250
 	0    1    1    0
@@
 P 1650 3350
 F 0 "C13" H 1850 3400 50  0000 L CNN
-F 1 "10 nF" V 1750 3250 50  0000 L CNN
+F 1 "1 nF" V 1750 3250 50  0000 L CNN
 F 2 "Capacitors_SMD:C_0402_NoSilk" H 1650 3350 50  0001 C CNN
 F 3 "" H 1650 3350 50  0001 C CNN
-F 4 " C15195" H 1650 3350 60  0001 C CNN "LCSC"
+F 4 "C1523" H 1650 3350 60  0001 C CNN "LCSC"
 	1    1650 3350
 	-1   0    0    1
@@
 P 3500 3950
 F 0 "C50" V 3350 3900 50  0000 L CNN
-F 1 "15 pF" V 3600 3900 50  0000 L CNN
+F 1 "1 pF" V 3600 3900 50  0000 L CNN
 F 2 "Capacitors_SMD:C_0402_NoSilk" H 3500 3950 50  0001 C CNN
 F 3 "" H 3500 3950 50  0001 C CNN
-F 4 "C1548" H 3500 3950 60  0001 C CNN "LCSC"
+F 4 "C14971" H 3500 3950 60  0001 C CNN "LCSC"
 	1    3500 3950
 	-1   0    0    1
@@
 P 4000 7050
 F 0 "C52" H 4010 7120 50  0000 L CNN
-F 1 "15 pF" V 3900 7000 50  0000 L CNN
+F 1 "1 pF" V 3900 7000 50  0000 L CNN
 F 2 "Capacitors_SMD:C_0402_NoSilk" H 4000 7050 50  0001 C CNN
 F 3 "" H 4000 7050 50  0001 C CNN
-F 4 "C1548" H 4000 7050 60  0001 C CNN "LCSC"
+F 4 "C14971" H 4000 7050 60  0001 C CNN "LCSC"
 	1    4000 7050
 	-1   0    0    1
